Commit message: Update quadx.xacro

File: urdf/quadx.xacro (robot description, xacro)
@@ -318,5 +318,5 @@
     <turnGravityOff>true</turnGravityOff>
   </gazebo>
-  <model>
+  <gazebo>
    <!--add lidar-->
         <link name="hokuyo_link">
@@ -374,5 +374,5 @@
             <plugin name="hokuyo_node" filename="libgazebo_ros_laser.so">
               <robotNamespace></robotNamespace>
-              <topicName>/spur/laser/scan</topicName>
+              <topicName>/quadx/laser/scan</topicName>
               <frameName>/hokuyo_sensor_link</frameName>
             </plugin>
@@ -384,4 +384,79 @@
           <child>hokuyo_link</child>
         </joint>
-  </model>
+  </gazebo>
+  <gazebo>
+     <link name="quadx_kinect_link">
+          <pose>0 0 0 0 0 0</pose>
+          <collision name="collision">
+            <pose>0 0 0.3 0 0 0</pose>
+            <geometry>
+              <box>
+                <size>0.1 0.1 0.1</size>
+              </box>
+            </geometry>
+          </collision>
+          <visual name="visual">
+            <pose>0 0 0.27 0 0 0</pose>
+            <geometry>
+              <mesh filename="package://quadx/snsr_dep/hokuyo.dae"/>
+            </geometry>
+          </visual>
+          <inertial>
+            <mass>0.016</mass>
+            <inertia>
+               <ixx>0.0001</ixx>
+               <ixy>0</ixy>
+               <ixz>0</ixz>
+               <iyy>0.0001</iyy>
+               <iyz>0</iyz>
+               <izz>0.0001</izz>
+               <!-- low intertia necessary to avoid not disturb the drone -->
+            </inertia>
+          </inertial>
+          <sensor name="quadx_kinect_camera" type="depth">
+            <update_rate>20</update_rate>
+            <camera>
+              <horizontal_fov>1.047198</horizontal_fov>
+              <image>
+                <width>640</width>
+                <height>480</height>
+                <format>R8G8B8</format>
+              </image>
+              <clip>
+                <near>0.05</near>
+                <far>3</far>
+              </clip>
+            </camera>
+            <plugin name="quadx_kinect_controller" filename="libgazebo_ros_openni_kinect.so">
+              <baseline>0.2</baseline>
+              <alwaysOn>true</alwaysOn>
+              <updateRate>1.0</updateRate>
+              <cameraName>quadx_kinect_ir</cameraName>
+              <imageTopicName>/quadx_kinect/color/image_raw</imageTopicName>
+              <cameraInfoTopicName>/quadx_kinect/color/camera_info</cameraInfoTopicName>
+              <depthImageTopicName>/quadx_kinect/depth/image_raw</depthImageTopicName>
+              <depthImageInfoTopicName>/quadx_kinect/depth/camera_info</depthImageInfoTopicName>
+              <pointCloudTopicName>/quadx_kinect/depth/points</pointCloudTopicName>
+              <frameName>quadx_kinect</frameName>
+              <pointCloudCutoff>0.5</pointCloudCutoff>
+              <pointCloudCutoffMax>3.0</pointCloudCutoffMax>
+              <distortionK1>0.00000001</distortionK1>
+              <distortionK2>0.00000001</distortionK2>
+              <distortionK3>0.00000001</distortionK3>
+              <distortionT1>0.00000001</distortionT1>
+              <distortionT2>0.00000001</distortionT2>
+              <CxPrime>0</CxPrime>
+              <Cx>0</Cx>
+              <Cy>0</Cy>
+              <focalLength>0</focalLength>
+              <hackBaseline>0</hackBaseline>
+            </plugin>
+          </sensor>
+        </link>
+        <joint name="my_kinect_joint" type="fixed">
+          <pose>0 0 0 0 0 0</pose>
+          <parent>base_link</parent>
+          <child>quadx_kinect_link</child>
+        </joint>
+  </gazebo>
 </robot>

Commit message: Update quadx.xacro

File: urdf/quadx.xacro (robot description, xacro)
@@ -455,5 +455,5 @@
           </sensor>
         </link>
-        <joint name="my_kinect_joint" type="fixed">
+        <joint name="quad_kinect_joint" type="fixed">
           <pose>0 0 0 0 0 0</pose>
           <parent>base_link</parent>
